Commit message: Port to Ubuntu 22.04, ROS 2 Humble and Gazebo Fortress
Humble's binary ros_gz and gz_ros2_control packages target Gazebo
Fortress, so the simulation is moved from Harmonic to Fortress:

- Use Fortress system plugin names in the URDF and worlds, load
  libgz_ros2_control-system.so, and downgrade worlds to SDF 1.9.
- Replace bullet-featherstone (unavailable in Fortress) with the
  default DART engine in default.sdf.
- Force gz_version 6 in the launch, set IGN_PARTITION alongside
  GZ_PARTITION and the Fortress resource path; clean_sim.sh also
  kills ign gazebo processes.
- Spawn the legs in the Go2 lying-down pose via ros2_control
  initial_value. The calf range excludes 0 and Fortress does not pull
  out-of-range joints back into limits, so starting at 0 made the calf
  chatter against its stop and flip the robot on the first stand.
- Update the README for Humble, joystick/BLE setup, and the branch.

File: unitree_go2_description/urdf/const.xacro (robot description, xacro)
@@ -53,4 +53,12 @@
     <xacro:property name="calf_velocity_max" value="20.06"/>
     <xacro:property name="calf_torque_max" value="35.55"/>
+    <!-- Initial joint pose: the Go2 lying-down pose. The calf range excludes 0,
+         and Gazebo Fortress does not pull a joint that spawns outside its
+         limits back into range, so starting at 0 makes the calf chatter
+         against its stop and flip the robot on the first stand. Spawning
+         folded also lets the passive robot settle flat on its belly. -->
+    <xacro:property name="initial_hip" value="0.0"/>
+    <xacro:property name="initial_thigh" value="1.36"/>
+    <xacro:property name="initial_calf" value="-2.65"/>
     <!-- dynamics inertial value -->
     <!-- trunk -->

File: unitree_go2_description/urdf/leg.xacro (robot description, xacro)
@@ -167,5 +167,5 @@
                 <contact>
                     <collision>${name}_lower_leg_link_fixed_joint_lump__${name}_foot_link_collision_1</collision>
-                    <!-- Gazebo Sim 8's Contact system reads topic here. -->
+                    <!-- Contact system (Fortress and Harmonic) reads topic here. -->
                     <topic>/feet/${contact_name}/contacts</topic>
                 </contact>
@@ -178,5 +178,7 @@
             <joint name="${name}_hip_joint">
                 <command_interface name="effort"/>
-                <state_interface name="position"/>
+                <state_interface name="position">
+                    <param name="initial_value">${initial_hip}</param>
+                </state_interface>
                 <state_interface name="velocity"/>
                 <state_interface name="effort"/>
@@ -184,5 +186,7 @@
             <joint name="${name}_upper_leg_joint">
                 <command_interface name="effort"/>
-                <state_interface name="position"/>
+                <state_interface name="position">
+                    <param name="initial_value">${initial_thigh}</param>
+                </state_interface>
                 <state_interface name="velocity"/>
                 <state_interface name="effort"/>
@@ -190,5 +194,7 @@
             <joint name="${name}_lower_leg_joint">
                 <command_interface name="effort"/>
-                <state_interface name="position"/>
+                <state_interface name="position">
+                    <param name="initial_value">${initial_calf}</param>
+                </state_interface>
                 <state_interface name="velocity"/>
                 <state_interface name="effort"/>

File: unitree_go2_description/urdf/unitree_go2_gazebo.xacro (robot description, xacro)
@@ -3,5 +3,5 @@
   <!-- Gazebo Sim plugins -->
   <gazebo>
-    <plugin filename="gz-sim-pose-publisher-system" name="gz::sim::systems::PosePublisher">
+    <plugin filename="ignition-gazebo-pose-publisher-system" name="ignition::gazebo::systems::PosePublisher">
       <publish_link_pose>true</publish_link_pose>
       <publish_sensor_pose>true</publish_sensor_pose>
@@ -16,5 +16,5 @@
   <!-- Robot-wide physics properties -->
   <!-- <gazebo>
-    <plugin filename="gz-sim-physics-system" name="gz::sim::systems::Physics">
+    <plugin filename="ignition-gazebo-physics-system" name="ignition::gazebo::systems::Physics">
       <engine>
         <filename>gz-physics-bullet-plugin</filename>
@@ -24,5 +24,5 @@
   <!-- ROS2 Control plugin -->
   <gazebo>
-    <plugin filename="gz_ros2_control-system" name="gz_ros2_control::GazeboSimROS2ControlPlugin">
+    <plugin filename="libgz_ros2_control-system.so" name="gz_ros2_control::GazeboSimROS2ControlPlugin">
       <parameters>$(find unitree_go2_sim)/config/ros_control/ros_control.yaml</parameters>
       <robot_param_node>robot_state_publisher</robot_param_node>
@@ -32,5 +32,5 @@
   <!-- Odometry plugin -->
   <gazebo>
-    <plugin filename="gz-sim-odometry-publisher-system" name="gz::sim::systems::OdometryPublisher">
+    <plugin filename="ignition-gazebo-odometry-publisher-system" name="ignition::gazebo::systems::OdometryPublisher">
       <!-- Publish the moving odom -> base_link transform.  The standard launch
            bridges this Gazebo Pose_V topic to ROS /tf for RViz and tf2. -->
@@ -93,5 +93,5 @@
         </linear_acceleration>
       </imu>
-      <plugin filename="gz-sim-imu-system" name="gz::sim::systems::Imu">
+      <plugin filename="ignition-gazebo-imu-system" name="ignition::gazebo::systems::Imu">
         <initial_orientation_as_reference>false</initial_orientation_as_reference>
       </plugin>
